File: dhere_mod_1.sch (KiCad schematic (older format))
At the start: 36 parts, among them J1 Power conn, J2 Input conn, J3 MOTOR, J4 Input conn, J5 Input conn, Q1 BC547, Q2 BC557, Q3 IRF4905, Q4 IRF3205, Q5 IRF4905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

Commit message: #2 fixed
Parts:
- added D4: LED, LED_THT:LED_D5.0mm_FlatTop, symbol Device:LED
- added R12: 5k, Resistor_SMD:R_0805_2012Metric_Pad1.15x1.40mm_HandSolder, symbol Device:R_Small
- added SW1: SW_SPDT, Button_Switch_THT:SW_CuK_OS102011MA1QN1_SPDT_Angled, symbol Switch:SW_SPDT
- Q1, Q2, Q7, Q8: footprint Package_TO_SOT_THT:TO-92_Inline -> Package_TO_SOT_THT:TO-92_Wide
- Q3, Q4, Q5, Q6: footprint Package_TO_SOT_THT:TO-220-3_Vertical -> kicad-library:TO-220-3_Vertical
- R1: footprint Resistor_THT:R_Axial_DIN0204_L3.6mm_D1.6mm_P5.08mm_Horizontal -> Resistor_SMD:R_0805_2012Metric_Pad1.15x1.40mm_HandSolder
- R10, R11, R2, R3, R4, R5, R6, R7, R8, R9: footprint Resistor_THT:R_Axial_DIN0204_L3.6mm_D1.6mm_P5.08mm_Horizontal -> Resistor_THT:R_Axial_DIN0207_L6.3mm_D2.5mm_P7.62mm_Horizontal
Connections:
- net GND: now also D4.1 (K); no longer J2.1 (Pin_1), J4.1 (Pin_1), J5.1 (Pin_1), U2.2, U3.2
- net VCC: now also C5.2, C6.2, Q3.3 (S), Q5.3 (S), SW1.3 (C); no longer J1.1 (Pin_1), Q3.2 (D), Q5.2 (D)
- net at J3.1 (Pin_1), Q6.2 (D): now also Q5.2 (D); no longer C5.2, Q5.3 (S)
- net at D2.2 (A), Q3.1 (G), Q4.1 (G)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: now also C6.1; no longer C6.2
- net at J3.2 (Pin_2), Q4.2 (D): now also Q3.2 (D); no longer C6.1, Q3.3 (S)
- new net: J1.1 (Pin_1), R12.2, SW1.1 (A), SW1.2 (B)
- new net: D4.2 (A), R12.1
- new net GNDD: J2.1 (Pin_1), J4.1 (Pin_1), J5.1 (Pin_1), U2.2, U3.2
Other:
- moved on the sheet: C5
